Commit message: revamped launch file

File: urdf-models/urdf/freya/ASV_MainAssembly.urdf (robot description, URDF)
Before this commit: robot ASV_MainAssembly, 1 links, 0 joints
Links:
- link base_link: mass 139.541646462225 -> None

Commit message: added base_link to base_link_ENU tf

File: urdf-models/urdf/freya/ASV_MainAssembly.urdf (robot description, URDF)
Before this commit: robot ASV_MainAssembly, 1 links, 0 joints
Links:
- removed link base_link
- added link base_link_ENU; collision mesh filename=package://urdf-models/meshes/base_link.STL; visual mesh filename=package://urdf-models/meshes/base_link.STL

Commit message: changed transform name

File: urdf-models/urdf/freya/ASV_MainAssembly.urdf (robot description, URDF)
Before this commit: robot ASV_MainAssembly, 1 links, 0 joints
Links:
- removed link base_link_ENU
- added link base_link_SEU; collision mesh filename=package://urdf-models/meshes/base_link.STL; visual mesh filename=package://urdf-models/meshes/base_link.STL

Commit message: renamed some stuff

File: urdf-models/urdf/freya/ASV_MainAssembly.urdf (robot description, URDF)
Before this commit: robot ASV_MainAssembly, 1 links, 0 joints
Links:
- link base_link_SEU: geometry collision mesh filename=package://urdf_models/meshes/freya.STL; visual mesh filename=package://urdf_models/meshes/freya.STL

Commit message: added launch file to launch urdf model and thruster viz

File: urdf-models/urdf/freya/ASV_MainAssembly.urdf (robot description, URDF)
Before this commit: robot ASV_MainAssembly, 1 links, 0 joints
Links:
- removed link base_link_SEU
- added link freya_model; collision mesh filename=package://urdf_models/meshes/freya.STL; visual mesh filename=package://urdf_models/meshes/freya.STL
